Commit message: feat: add MuJoCo support and launch files for xArm7 integration

File: xarm_description/urdf/xarm7/xarm7.ros2_control.xacro (robot description, xacro)
@@ -1,5 +1,6 @@
 <?xml version="1.0"?>
 <robot xmlns:xacro="http://ros.org/wiki/xacro">
-  <xacro:macro name="xarm7_ros2_control" params="prefix
+  <xacro:macro name="xarm7_ros2_control"
+    params="prefix
     velocity_control:='false'
     ros2_control_plugin:='uf_robot_hardware/UFRobotSystemHardware'
@@ -29,4 +30,9 @@
           <param name="add_bio_gripper">${add_bio_gripper}</param>
         </xacro:if>
+        <xacro:if value="${ros2_control_plugin == 'mujoco_ros2_simulation/MujocoSystemInterface'}">
+          <!-- Add MuJoCo specific parameters here if needed -->
+          <param name="mujoco_model">$(find mujoco_ros2_simulation)/resources/scene_xarm7.xml</param>
+          <param name="headless">false</param>
+        </xacro:if>
       </hardware>
       <joint name="${prefix}joint1">
@@ -39,6 +45,6 @@
           <param name="max">3.14</param>
         </command_interface>
-        <state_interface name="position"/>
-        <state_interface name="velocity"/>
+        <state_interface name="position" />
+        <state_interface name="velocity" />
         <!-- <state_interface name="effort"/> -->
       </joint>
@@ -52,6 +58,6 @@
           <param name="max">3.14</param>
         </command_interface>
-        <state_interface name="position"/>
-        <state_interface name="velocity"/>
+        <state_interface name="position" />
+        <state_interface name="velocity" />
         <!-- <state_interface name="effort"/> -->
       </joint>
@@ -65,6 +71,6 @@
           <param name="max">3.14</param>
         </command_interface>
-        <state_interface name="position"/>
-        <state_interface name="velocity"/>
+        <state_interface name="position" />
+        <state_interface name="velocity" />
         <!-- <state_interface name="effort"/> -->
       </joint>
@@ -78,6 +84,6 @@
           <param name="max">3.14</param>
         </command_interface>
-        <state_interface name="position"/>
-        <state_interface name="velocity"/>
+        <state_interface name="position" />
+        <state_interface name="velocity" />
         <!-- <state_interface name="effort"/> -->
       </joint>
@@ -91,6 +97,6 @@
           <param name="max">3.14</param>
         </command_interface>
-        <state_interface name="position"/>
-        <state_interface name="velocity"/>
+        <state_interface name="position" />
+        <state_interface name="velocity" />
         <!-- <state_interface name="effort"/> -->
       </joint>
@@ -104,6 +110,6 @@
           <param name="max">3.14</param>
         </command_interface>
-        <state_interface name="position"/>
-        <state_interface name="velocity"/>
+        <state_interface name="position" />
+        <state_interface name="velocity" />
         <!-- <state_interface name="effort"/> -->
       </joint>
@@ -117,6 +123,6 @@
           <param name="max">3.14</param>
         </command_interface>
-        <state_interface name="position"/>
-        <state_interface name="velocity"/>
+        <state_interface name="position" />
+        <state_interface name="velocity" />
         <!-- <state_interface name="effort"/> -->
       </joint>
